File: rf_noise_antenna.sch (KiCad schematic (older format))
At the start: 31 parts

Commit message: adding com Values
Parts:
- added J?: Conn_01x03, symbol Conn_01x03
- C? (x2): value C -> 100nF
- C? (x2): value CP -> 4.7uF 16V
- C?: value CP -> 47uF 16V
- D? (x2): value D -> 4148
- R?: value R -> 1k2
- R?: value R -> 250
Connections:
- wire segments 64 -> 84
Other:
- note added: "12V Powersupply for\n Active Antenna"
- note added: "HPF"
- note added: "LPF"
- note added: "RF from Sctive Antenna"
- note added: "RF to SDR Dongle"
- moved on the sheet: C?

Commit message: Change isolation to be at antenna
Parts:
- removed J?: Conn_01x02, symbol Conn_01x02
- removed J?: Conn_01x03, symbol Conn_01x03
- removed T?: Transformer_1P_1S, symbol Transformer_1P_1S
- added J?: Conn_01x03, symbol Conn_01x03
- added T?: Transformer_1P_1S, symbol Transformer_1P_1S
Connections:
- wire segments 84 -> 65
Other:
- moved on the sheet: C?, D?, J?, L?, Q?, R?, U?

Commit message: Fix DR cherck
Parts:
- gave numbers to parts that had none: 31
Connections:
- wire segments 65 -> 81
- no-connect marks 0 -> 29
Other:
- moved on the sheet: C1, C2, C7, C8, L4, L5, L6

Commit message: Replace relay with Solit state
Parts:
- removed D1, D2: 4148, symbol D
- removed K1, K2: FINDER-32.21-x000, Relays_THT:Relay_SPST_Finder_32.21-x300, symbol FINDER-32.21-x000
- added C? (x4): 100nF, symbol C
- added K? (x2): MASWSS0115, RF_switch:SPDT, symbol MASWSS0115
- added Q?: 2N2219, TO_SOT_Packages_THT:TO-39-3, symbol 2N2219
- added R?: 1k2, symbol R
- added R? (x2): 250, symbol R
Connections:
- net labels added: +5V
- wire segments 81 -> 92
- no-connect marks 29 -> 28
Other:
- moved on the sheet: C1, C10, C11, C2, C4, C5, C6, D3, J2, J4, L1, L2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

Commit message: add componet ref
Parts:
- removed T1: Transformer_1P_1S, symbol Transformer_1P_1S
- added T1: MABA-009180-500MHz_1P_1S, symbol MABA-009180-500MHz_1P_1S
- C1, C2, C6, C7: renamed from C?; footprint (none) -> Capacitors_SMD:C_0805_HandSoldering
- C10: renamed from C6; value C -> 390pF; footprint (none) -> Capacitors_SMD:C_0805_HandSoldering
- C11: renamed from C9; footprint (none) -> Capacitors_SMD:C_0805_HandSoldering
- C14: renamed from C10; footprint (none) -> Capacitors_SMD:C_0805_HandSoldering
- C3: renamed from C1; value C -> 360pF; footprint (none) -> Capacitors_SMD:C_0805_HandSoldering
- C4: renamed from C2; value C -> 360pF; footprint (none) -> Capacitors_SMD:C_0805_HandSoldering
- C5: renamed from C3; value C -> 100nF; footprint (none) -> Capacitors_SMD:C_0805_HandSoldering
- C8: renamed from C4; value C -> 390pF; footprint (none) -> Capacitors_SMD:C_0805_HandSoldering
- C9: renamed from C5; value C -> 120pF; footprint (none) -> Capacitors_SMD:C_0805_HandSoldering
- D1: renamed from D3; footprint (none) -> LEDs:LED_0805_HandSoldering
- J1, J2: footprint (none) -> Connectors_Molex:Molex_SMA_Jack_Edge_Mount
- J3: footprint (none) -> Connectors_Terminal_Blocks:TerminalBlock_Philmore_TB133_03x5mm_Straight
- L1, L3: value L -> 330nH; footprint (none) -> Inductors_SMD:L_0805_HandSoldering
- L2: value L -> 1.1uH; footprint (none) -> Inductors_SMD:L_0805_HandSoldering
- L4: value L -> 1mH; footprint (none) -> Inductors_SMD:L_0805_HandSoldering
- L5, L6: value L -> 360nH; footprint (none) -> Inductors_SMD:L_0805_HandSoldering
- R1, R2, R3: renamed from R?; footprint (none) -> Resistors_SMD:R_0805_HandSoldering
- R4: renamed from R1; footprint (none) -> Resistors_SMD:R_0805_HandSoldering
- R5: renamed from R2; footprint (none) -> Resistors_SMD:R_0805_HandSoldering
- U1: footprint (none) -> Power_Integrations:TO-220
- gave numbers to parts that had none: 3
- renumbered C7 to C12, C8 to C13, C11 to C15, Q1 to Q2
Connections:
- net GND: now also T1.4 (SB)
- net GNDA: now also T1.3 (SA)
- net at C5.1: now also T1.1 (AA)
- net at C6.2: now also T1.5 (S)
- no-connect marks 28 -> 31
Other:
- note added: "High Pass filter (14.2Mhz)"
- note added: "Low Pass Filter (14.2Mhz)"
- note removed: "HPF"
- note removed: "LPF"
- moved on the sheet: C1, C10, C11, C12, C13, C14, C15, C2, C3, C4, C5, C6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

Commit message: Starting with PCB Layout
Parts:
- added H1, H2, H3, H4: Conn_01x01, Mounting_Holes:MountingHole_3.2mm_M3, symbol Conn_01x01
- C12: footprint (none) -> Capacitors_Tantalum_SMD:CP_Tantalum_Case-C_EIA-6032-28_Hand
- C13, C15: footprint (none) -> Capacitors_SMD:C_0805_HandSoldering
- K1, K2: footprint RF_switch:SPDT -> rf_noise_antenna:SC-70-6
- Q1, Q2: value 2N2219 -> BC817; footprint TO_SOT_Packages_THT:TO-39-3 -> TO_SOT_Packages_SMD:SOT-23
- T1: footprint (none) -> rf_noise_antenna:SM22
- U1: footprint Power_Integrations:TO-220 -> TO_SOT_Packages_THT:TO-220_Horizontal
Connections:
- net GND: now also H1.1 (Pin_1), H2.1 (Pin_1), H3.1 (Pin_1), H4.1 (Pin_1)
- no-connect marks 31 -> 30
Changed lines of the file:
@@
 P 9750 2700
 F 0 "Q2" H 9950 2775 50  0000 L CNN
-F 1 "2N2219" H 9950 2700 50  0000 L CNN
-F 2 "TO_SOT_Packages_THT:TO-39-3" H 9950 2625 50  0001 L CIN
+F 1 "BC817" H 9950 2700 50  0000 L CNN
+F 2 "TO_SOT_Packages_SMD:SOT-23" H 9950 2625 50  0001 L CIN
 F 3 "" H 9750 2700 50  0001 L CNN
 	1    9750 2700
@@
 F 0 "C15" H 6825 3000 50  0000 L CNN
 F 1 "4.7uF 16V" H 6600 2800 50  0000 L CNN
-F 2 "" H 6838 2750 50  0001 C CNN
+F 2 "Capacitors_SMD:C_0805_HandSoldering" H 6838 2750 50  0001 C CNN
 F 3 "" H 6800 2900 50  0001 C CNN
 	1    6800 2900
@@
 U 1 1 5B76CCF1
 P 3250 1450
-F 0 "L4" H 3200 1450 50  0000 C CNN
+F 0 "L4" H 3150 1450 50  0000 C CNN
 F 1 "1mH" V 3325 1450 50  0000 C CNN
 F 2 "Inductors_SMD:L_0805_HandSoldering" H 3250 1450 50  0001 C CNN
@@
 F 0 "C13" H 3175 2350 50  0000 L CNN
 F 1 "4.7uF 16V" H 3175 2150 50  0000 L CNN
-F 2 "" H 3188 2100 50  0001 C CNN
+F 2 "Capacitors_SMD:C_0805_HandSoldering" H 3188 2100 50  0001 C CNN
 F 3 "" H 3150 2250 50  0001 C CNN
 	1    3150 2250
@@
 F 0 "U1" H 2550 2125 50  0000 C CNN
 F 1 "L7809" H 2700 2125 50  0000 L CNN
-F 2 "Power_Integrations:TO-220" H 2725 1850 50  0001 L CIN
+F 2 "TO_SOT_Packages_THT:TO-220_Horizontal" H 2725 1850 50  0001 L CIN
 F 3 "" H 2700 1950 50  0001 C CNN
 	1    2700 2000
@@
 F 0 "C12" H 2225 2350 50  0000 L CNN
 F 1 "47uF 16V" H 2225 2150 50  0000 L CNN
-F 2 "" H 2238 2100 50  0001 C CNN
+F 2 "Capacitors_Tantalum_SMD:CP_Tantalum_Case-C_EIA-6032-28_Hand" H 2238 2100 50  0001 C CNN
 F 3 "" H 2200 2250 50  0001 C CNN
 	1    2200 2250
@@
 12V Powersupply for\n Active Antenna
 Wire Wire Line
-	6750 850  6900 850
-Wire Wire Line
-	6900 850  7000 850
-Wire Wire Line
-	7300 850  7400 850
-Wire Wire Line
-	7400 850  7550 850
-Wire Wire Line
-	6800 1600 6900 1600
-Wire Wire Line
-	6900 1600 7000 1600
-Wire Wire Line
-	7300 1600 7450 1600
-Wire Wire Line
-	7450 1600 7600 1600
+	6750 850  7000 850
+Wire Wire Line
+	7300 850  7550 850
+Wire Wire Line
+	6800 1600 7000 1600
+Wire Wire Line
+	7300 1600 7600 1600
 Wire Wire Line
 	7900 1600 7900 1350
@@
 	10050 1450 10050 1700
 Wire Wire Line
-	7150 2750 7150 3000
-Wire Wire Line
-	7150 3000 7150 3350
+	7150 2750 7150 3350
 Connection ~ 6800 2750
 Connection ~ 6550 2750
@@
 Connection ~ 7150 3000
 Wire Wire Line
-	3000 1200 3250 1200
-Wire Wire Line
-	3250 1200 3350 1200
+	3000 1200 3350 1200
 Wire Wire Line
 	2850 1400 2850 1500
 Wire Wire Line
-	3000 2000 3150 2000
-Wire Wire Line
-	3150 2000 3250 2000
-Wire Wire Line
-	3250 2000 3400 2000
-Wire Wire Line
-	3250 1600 3250 1750
-Wire Wire Line
-	3250 1750 3250 2000
+	3000 2000 3400 2000
+Wire Wire Line
+	3250 1600 3250 2000
 Connection ~ 3250 2000
 Wire Wire Line
@@
 	6550 3050 6550 3150
 Wire Wire Line
-	6550 3150 6650 3150
-Wire Wire Line
-	6650 3150 6800 3150
+	6550 3150 6800 3150
 Wire Wire Line
 	6800 3150 6800 3050
@@
 	6850 5950 6850 6250
 Wire Wire Line
-	6850 6250 6950 6250
-Wire Wire Line
-	6950 6250 7050 6250
-Wire Wire Line
-	7050 6250 7150 6250
-Wire Wire Line
-	7150 6250 7250 6250
-Wire Wire Line
-	7250 6250 7350 6250
-Wire Wire Line
-	7350 6250 7450 6250
-Wire Wire Line
-	7450 6250 7550 6250
+	6850 6250 7550 6250
 Wire Wire Line
 	6950 5950 6950 6250
@@
 Connection ~ 7050 6250
 Wire Wire Line
-	7150 5950 7150 6250
-Wire Wire Line
-	7150 6250 7150 6350
+	7150 5950 7150 6350
 Wire Wire Line
 	7250 6250 7250 5950
@@
 F 0 "K1" V 5150 1150 50  0000 L CNN
 F 1 "MASWSS0115" V 5900 1150 50  0000 C CNN
-F 2 "RF_switch:SPDT" H 5500 1800 50  0001 C CNN
+F 2 "rf_noise_antenna:SC-70-6" H 5500 1800 50  0001 C CNN
 F 3 "" H 5350 1150 50  0001 C CNN
 	1    5500 1150
@@
 F 0 "K2" V 8500 1200 50  0000 L CNN
 F 1 "MASWSS0115" V 9250 1200 50  0000 C CNN
-F 2 "RF_switch:SPDT" H 8850 1850 50  0001 C CNN
+F 2 "rf_noise_antenna:SC-70-6" H 8850 1850 50  0001 C CNN
 F 3 "" H 8700 1200 50  0001 C CNN
 	1    8850 1200
@@
 $EndComp
 Wire Wire Line
-	6300 2750 6550 2750
-Wire Wire Line
-	6550 2750 6800 2750
-Wire Wire Line
-	6800 2750 7150 2750
+	6300 2750 7150 2750
 $Comp
 L +5V #PWR020
@@
 P 5600 2450
 F 0 "Q1" H 5800 2525 50  0000 L CNN
-F 1 "2N2219" H 5800 2450 50  0000 L CNN
-F 2 "TO_SOT_Packages_THT:TO-39-3" H 5800 2375 50  0001 L CIN
+F 1 "BC817" H 5800 2450 50  0000 L CNN
+F 2 "TO_SOT_Packages_SMD:SOT-23" H 5800 2375 50  0001 L CIN
 F 3 "" H 5600 2450 50  0001 L CNN
 	1    5600 2450
@@
 $EndComp
 Wire Wire Line
-	9850 2400 9850 2450
-Wire Wire Line
-	9850 2450 9850 2500
+	9850 2400 9850 2500
 Wire Wire Line
 	9850 2000 9850 2100
@@
 	9350 1050 9450 1050
 Wire Wire Line
-	9450 600  9450 1050
-Wire Wire Line
-	9450 1050 9450 2450
-Wire Wire Line
-	9450 2450 9850 2450
-Wire Wire Line
-	9850 2450 10100 2450
+	9450 600  9450 2450
+Wire Wire Line
+	9450 2450 10100 2450
 Connection ~ 9850 2450
 Wire Wire Line
@@
 $EndComp
 Wire Wire Line
-	5500 2150 5500 2200
-Wire Wire Line
-	5500 2200 5500 2250
+	5500 2150 5500 2250
 $Comp
 L GND #PWR023
@@
 	5500 2650 5500 2750
 Wire Wire Line
-	4900 2200 5500 2200
-Wire Wire Line
-	5500 2200 9350 2200
+	4900 2200 9350 2200
 Wire Wire Line
 	4900 2200 4900 1400
@@
 	7400 1200 7400 1250
 Wire Wire Line
-	1900 2000 2200 2000
-Wire Wire Line
-	2200 2000 2400 2000
+	1900 2000 2400 2000
 Wire Wire Line
 	2700 2300 2700 2400
@@
 F 0 "T1" H 4150 1650 50  0000 C CNN
 F 1 "MABA-009180-500MHz_1P_1S" H 4150 1750 50  0000 C CNN
-F 2 "" H 4150 1400 50  0001 C CNN
+F 2 "rf_noise_antenna:SM22" H 4150 1400 50  0001 C CNN
 F 3 "" H 4150 1400 50  0001 C CNN
 	1    4150 1400
@@
 NoConn ~ 3750 1400
 NoConn ~ 3900 750
-NoConn ~ 3200 1450
+$Comp
+L Conn_01x01 H1
+U 1 1 5B7FB208
+P 2400 3450
+F 0 "H1" H 2400 3550 50  0000 C CNN
+F 1 "Conn_01x01" H 2400 3350 50  0000 C CNN
+F 2 "Mounting_Holes:MountingHole_3.2mm_M3" H 2400 3450 50  0001 C CNN
+F 3 "" H 2400 3450 50  0001 C CNN
+	1    2400 3450
+	1    0    0    -1
+$EndComp
+$Comp
+L Conn_01x01 H2
+U 1 1 5B7FB2FF
+P 2400 3750
+F 0 "H2" H 2400 3850 50  0000 C CNN
+F 1 "Conn_01x01" H 2400 3650 50  0000 C CNN
+F 2 "Mounting_Holes:MountingHole_3.2mm_M3" H 2400 3750 50  0001 C CNN
+F 3 "" H 2400 3750 50  0001 C CNN
+	1    2400 3750
+	1    0    0    -1
+$EndComp
+$Comp
+L Conn_01x01 H3
+U 1 1 5B7FB413
+P 2400 4000
+F 0 "H3" H 2400 4100 50  0000 C CNN
+F 1 "Conn_01x01" H 2400 3900 50  0000 C CNN
+F 2 "Mounting_Holes:MountingHole_3.2mm_M3" H 2400 4000 50  0001 C CNN
+F 3 "" H 2400 4000 50  0001 C CNN
+	1    2400 4000
+	1    0    0    -1
+$EndComp
+$Comp
+L Conn_01x01 H4
+U 1 1 5B7FB4A1
+P 2400 4300
+F 0 "H4" H 2400 4400 50  0000 C CNN
+F 1 "Conn_01x01" H 2400 4200 50  0000 C CNN
+F 2 "Mounting_Holes:MountingHole_3.2mm_M3" H 2400 4300 50  0001 C CNN
+F 3 "" H 2400 4300 50  0001 C CNN
+	1    2400 4300
+	1    0    0    -1
+$EndComp
+$Comp
+L GND #PWR024
+U 1 1 5B7FC079
+P 1400 4000
+F 0 "#PWR024" H 1400 3750 50  0001 C CNN
+F 1 "GND" H 1400 3850 50  0000 C CNN
+F 2 "" H 1400 4000 50  0001 C CNN
+F 3 "" H 1400 4000 50  0001 C CNN
+	1    1400 4000
+	1    0    0    -1
+$EndComp
+Wire Wire Line
+	2200 3450 1400 3450
+Wire Wire Line
+	1400 3450 1400 4000
+Wire Wire Line
+	2200 3750 1400 3750
+Connection ~ 1400 3750
+Wire Wire Line
+	2200 4000 1850 4000
+Wire Wire Line
+	1850 4000 1850 3750
+Connection ~ 1850 3750
+Wire Wire Line
+	2200 4300 1750 4300
+Wire Wire Line
+	1750 4300 1750 3750
+Connection ~ 1750 3750
 $EndSCHEMATC
