File: _saved_rf_noise_antenna.sch (KiCad schematic (older format))
At the start: 41 parts, among them J1 Conn_Coaxial, J2 Conn_Coaxial, J3 Conn_01x03, J4 Raspberry_Pi_2_3, K1 MASWSS0115, K2 MASWSS0115, Q1 BC817, Q2 BC817, T1 MABA-009180-500MHz_1P_1S, U1 L7809

Commit message: Compleet pcb
Connections:
- net at C11.1, C13.1, L4.2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: now also J3.2 (Pin_2); no longer J3.3 (Pin_3)
- net at C12.1, U1.1 (IN): now also J3.3 (Pin_3); no longer J3.2 (Pin_2)
Other:
- note added: "12V Power supply \nfor Active Antenna"
- note removed: "12V Powersupply for\n Active Antenna"
Changed lines of the file:
@@
 Text Notes 6650 700  0    60   ~ 0
 Low Pass Filter (14.2Mhz)
-Text Notes 10350 1250 0    60   ~ 0
+Text Notes 10200 1250 0    60   ~ 0
 RF to SDR Dongle
 Text Notes 1250 1200 0    60   ~ 0
 RF from Sctive Antenna.\n9V Injection
-Text Notes 300  2150 0    60   ~ 0
-12V Powersupply for\n Active Antenna
+Text Notes 450  2050 0    60   ~ 0
+12V Power supply \nfor  Active Antenna
 $Comp
 L GND #PWR09
@@
 	3350 1200 3450 1200
 Wire Wire Line
-	1600 1900 1850 1900
-Wire Wire Line
-	1850 1900 1850 1750
-Wire Wire Line
-	1850 1750 2950 1750
+	1750 1750 2950 1750
 Connection ~ 2950 1750
 Wire Wire Line
-	1900 2100 1900 2000
+	1900 1900 1900 2100
 Connection ~ 1900 2000
 Wire Wire Line
@@
 	7400 1200 7400 1250
 Wire Wire Line
-	1600 2000 2100 2000
-Wire Wire Line
 	2400 2300 2400 2400
 Wire Wire Line
@@
 Wire Wire Line
 	5000 600  5000 1000
+Wire Wire Line
+	1750 1750 1750 2000
+Wire Wire Line
+	1750 2000 1600 2000
+Wire Wire Line
+	1600 1900 1900 1900
+Wire Wire Line
+	1900 2000 2100 2000
 $EndSCHEMATC
