File: _autosave-rf_noise_antenna_v2.kicad_pcb (KiCad board)
At the start: 2 copper layers, 65 x 56.5 mm, 41 parts, among them J1 Conn_Coaxial, J2 Conn_Coaxial, J3 Conn_01x03, J4 Raspberry_Pi_2_3, K1 MASWSS0115, K2 MASWSS0115, Q1 BC847, Q2 BC847, T1 MABA-009180-500MHz_1P_1S, U1 L7809

Commit message: adding V2 files
Parts:
- added D2: LED, LEDs:LED_0805_HandSoldering, F.Cu at (55.2, 67.2)
- added R6: 250, Resistors_SMD:R_0805_HandSoldering, F.Cu at (58.2, 67.2)
- added REF**: MountingHole_3.2mm_M3, Mounting_Holes:MountingHole_3.2mm_M3, F.Cu at (90.0, 36.8)
- added REF**: MountingHole_3.2mm_M3, Mounting_Holes:MountingHole_3.2mm_M3, F.Cu at (77.5, 36.8)
- added REF**: MountingHole_3.2mm_M3, Mounting_Holes:MountingHole_3.2mm_M3, F.Cu at (76.7, 53.8)
- added REF**: MountingHole_3.2mm_M3, Mounting_Holes:MountingHole_3.2mm_M3, F.Cu at (90.0, 53.8)
- J1, J2: footprint Connectors_Molex:Molex_SMA_Jack_Edge_Mount -> Bacar:SMA_Edge
- L4: value 1mH -> 10uH
- U1: value L7809 -> L7812
- moved J2 2.16 mm to (61.5, 74.5), turned to 180 degrees
- moved J1 1.90 mm to (31.6, 34.5), turned to 90 degrees
Connections:
- D1 pad 1: GND -> Net-(D1-Pad1)
- J4 pad 1: (no net) -> Net-(J4-Pad1)
- J4 pad 10: (no net) -> Net-(J4-Pad10)
- J4 pad 11: (no net) -> Net-(J4-Pad11)
- J4 pad 12: (no net) -> Net-(J4-Pad12)
- J4 pad 13: (no net) -> Net-(J4-Pad13)
- J4 pad 15: (no net) -> Net-(J4-Pad15)
- J4 pad 16: (no net) -> Net-(J4-Pad16)
- J4 pad 17: (no net) -> Net-(J4-Pad17)
- J4 pad 18: (no net) -> Net-(J4-Pad18)
- J4 pad 19: (no net) -> Net-(J4-Pad19)
- J4 pad 21: (no net) -> Net-(J4-Pad21)
- J4 pad 22: (no net) -> Net-(J4-Pad22)
- J4 pad 23: (no net) -> Net-(J4-Pad23)
- J4 pad 24: (no net) -> Net-(J4-Pad24)
- J4 pad 26: (no net) -> Net-(J4-Pad26)
- J4 pad 27: (no net) -> Net-(J4-Pad27)
- J4 pad 28: (no net) -> Net-(J4-Pad28)
- J4 pad 29: (no net) -> Net-(J4-Pad29)
- J4 pad 31: (no net) -> Net-(J4-Pad31)
- J4 pad 32: (no net) -> Net-(J4-Pad32)
- J4 pad 33: (no net) -> Net-(J4-Pad33)
- J4 pad 35: (no net) -> Net-(J4-Pad35)
- J4 pad 36: (no net) -> Net-(J4-Pad36)
- J4 pad 37: (no net) -> Net-(J4-Pad37)
- J4 pad 38: (no net) -> Net-(J4-Pad38)
- J4 pad 40: (no net) -> Net-(J4-Pad40)
- J4 pad 7: (no net) -> Net-(J4-Pad7)
- J4 pad 8: (no net) -> Net-(J4-Pad8)
- K1 pad 4: Net-(K1-Pad4) -> Net-(D1-Pad1)
- K2 pad 6: Net-(K1-Pad4) -> Net-(D1-Pad1)
- Q2 pad 3: Net-(K1-Pad4) -> Net-(D1-Pad1)
- R2 pad 1: Net-(K1-Pad4) -> Net-(D1-Pad1)
- R4 pad 2: Net-(K1-Pad4) -> +5V
- T1 pad 2: (no net) -> Net-(T1-Pad2)
Routing:
- net Net-(K1-Pad4): track 69.6 -> 0.00 mm
- net Net-(D1-Pad1): track 0.00 -> 65.0 mm
- net +5V: track 31.9 -> 94.5 mm, vias 1 -> 3
- net GND: track 396.5 -> 418.3 mm, vias 42 -> 51
- net Net-(D2-Pad2): track 0.00 -> 2.92 mm
- net Net-(D2-Pad1): track 59.5 -> 61.5 mm
Other:
- board text added: "ANT"
- board text added: "RF Isolation with Low and High Pass filter"
- board text added: "RF Noise Raspberry Hat V1.2"
- board text added: "RTL Rreceiver"
- board text added: "RX"
- board text removed: "RF Noise Raspberry Hat V1.0"
