File: rf_noise_antenna.kicad_pcb (KiCad board)
At the start: 2 copper layers, 65 x 56.5 mm, 41 parts, among them J1 Conn_Coaxial, J2 Conn_Coaxial, J3 Conn_01x03, J4 Raspberry_Pi_2_3, K1 MASWSS0115, K2 MASWSS0115, Q1 BC817, Q2 BC817, T1 MABA-009180-500MHz_1P_1S, U1 L7809

Commit message: Starting with PCB Layout
Parts:
- moved J3 49.2 mm to (39.4, 71.8), turned to 0 degrees
- moved C12 47.6 mm to (32.5, 64.5)
- moved C13 44.9 mm to (37.8, 42.2), turned to 90 degrees
- moved C11 41.1 mm to (42.2, 38.4), turned to 0 degrees
- moved U1 28.4 mm to (45.7, 42.2), turned to 180 degrees
- moved C6 19.0 mm to (57.9, 34.5)
- moved C5 17.6 mm to (51.3, 34.5)
- moved K1 17.5 mm to (60.5, 36.1)
- moved C2 16.9 mm to (66.0, 59.9)
- moved L3 16.9 mm to (66.0, 54.9)
- moved T1 16.8 mm to (55.9, 38.1), turned to 0 degrees
- moved C8 16.6 mm to (57.4, 45.7)
- moved L5 16.5 mm to (55.9, 49.3)
- moved L2 16.5 mm to (66.0, 46.7)
- moved C4 16.5 mm to (67.1, 50.8)
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Other:
- outline, holes or cut-outs redrawn

Commit message: Compleet pcb
Parts:
- moved R5 22.6 mm to (47.0, 30.2), turned to 90 degrees
- moved Q1 17.0 mm to (43.4, 30.5), turned to 270 degrees
- moved R1 16.4 mm to (55.9, 29.5), turned to 0 degrees
- moved C14 14.8 mm to (62.5, 30.7), turned to 90 degrees
- moved C15 14.1 mm to (59.7, 30.7), turned to 90 degrees
- moved Q2 13.7 mm to (50.8, 30.7), turned to 270 degrees
- moved R2 13.7 mm to (55.9, 31.8)
- moved C5 9.91 mm to (41.4, 34.8)
- moved T1 8.44 mm to (47.8, 35.8)
- moved R3 7.03 mm to (39.9, 30.5), turned to 270 degrees
- moved C6 6.13 mm to (51.9, 35.9), turned to 90 degrees
- moved K1 4.93 mm to (55.6, 37.1), turned to 180 degrees
- moved D1 3.19 mm to (67.4, 65.0)
- moved R4 2.71 mm to (67.3, 67.6)
- moved L6 2.30 mm to (58.2, 56.6), turned to 180 degrees
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Connections:
- J3 pad 2: Net-(C12-Pad1) -> Net-(C11-Pad1)
- J3 pad 3: Net-(C11-Pad1) -> Net-(C12-Pad1)
- J4 pad 10: Net-(J4-Pad10) -> (no net)
- J4 pad 3: (no net) -> Net-(J4-Pad3)
- J4 pad 5: (no net) -> Net-(J4-Pad5)
- J4 pad 8: Net-(J4-Pad8) -> (no net)
- K1 pad 1: Net-(C1-Pad2) -> Net-(C8-Pad2)
- K1 pad 3: Net-(C8-Pad2) -> Net-(C1-Pad2)
- K2 pad 4: Net-(K1-Pad4) -> Net-(K1-Pad6)
- K2 pad 6: Net-(K1-Pad6) -> Net-(K1-Pad4)
- Q1 pad 3: Net-(K1-Pad4) -> Net-(K1-Pad6)
- Q2 pad 3: Net-(K1-Pad6) -> Net-(K1-Pad4)
- R1 pad 1: Net-(K1-Pad4) -> Net-(K1-Pad6)
- R2 pad 1: Net-(K1-Pad6) -> Net-(K1-Pad4)
- R3 pad 1: Net-(J4-Pad8) -> Net-(J4-Pad3)
- R4 pad 2: Net-(K1-Pad6) -> Net-(K1-Pad4)
- R5 pad 2: Net-(J4-Pad10) -> Net-(J4-Pad5)
Routing:
- net GND: track 1.41 -> 409.3 mm, vias 0 -> 41
- net GNDA: track 0.00 -> 80.6 mm, vias 0 -> 3
- net Net-(K1-Pad4): track 0.00 -> 69.6 mm
- net Net-(K1-Pad6): track 0.00 -> 59.1 mm
- net Net-(C12-Pad1): track 0.00 -> 55.4 mm
- net Net-(C11-Pad1): track 0.00 -> 43.3 mm
- net +5V: track 0.00 -> 31.9 mm, vias 0 -> 1
- net Net-(C5-Pad2): track 0.00 -> 8.45 mm
- net Net-(C1-Pad2): track 0.00 -> 7.86 mm
- net Net-(C8-Pad2): track 0.00 -> 6.76 mm
- net Net-(J4-Pad5): track 0.00 -> 5.62 mm
- net Net-(C10-Pad2): track 0.00 -> 5.48 mm
- net Net-(C4-Pad2): track 0.00 -> 5.19 mm
- net Net-(C7-Pad1): track 0.00 -> 4.79 mm
- net Net-(C8-Pad1): track 0.00 -> 4.76 mm
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- added copper zone on B.Cu, net GND
- added copper zone on F.Cu, net GND
- added copper zone on B.Cu, net GNDA
- added copper zone on F.Cu, net GNDA
Other:
- net class +5V added: clearance 0.15, trace_width 0.5, via_dia 0.889, via_drill 0.381
- net class Default: clearance 0.254 -> 0.2
- net class GND added: clearance 0.15, trace_width 0.4, via_dia 0.889, via_drill 0.381
- net class Rf: clearance 0.254 -> 0.25; trace_width 1 -> 1.25
- net class Slim_rf added: clearance 0.1, trace_width 0.4, via_dia 0.889, via_drill 0.381
- rule trace_clearance: 0.254 -> 0.2

Commit message: Added measurmets
Routing:
- net GNDA: track 80.6 -> 126.0 mm, vias 3 -> 24
Other:
- board text added: "Giga Technology"
- board text added: "RF Noise Raspberry Hat V1.0"
- board text added: "http://www.giga.co.za"
Changed lines of the file:
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@@
     (area 16.276381 15.477 105.89762 87.217001)
     (thickness 1.6)
-    (drawings 38)
-    (tracks 363)
+    (drawings 41)
+    (tracks 411)
     (zones 0)
     (modules 41)
@@
   (title_block
     (title "RaspberryPi Hat Board")
+    (date 2018-08-26)
     (rev 1)
-    (company disk91.com)
-    (comment 1 "(c) Paul Pinault 2015")
-    (comment 2 "(c) Disk91")
+    (company "Giga Technology")
+    (comment 1 "RF Noise Pi Hat")
+    (comment 2 "Author: Anton Janovsky")
   )
   (layers
@@
     (trace_clearance 0.2)
     (zone_clearance 0.508)
-    (zone_45_only no)
+    (zone_45_only yes)
     (trace_min 0.254)
     (segment_width 0.2)
@@
     )
   )
+  (gr_text http://www.giga.co.za (at 83.7565 37.6555) (layer F.SilkS)
+    (effects (font (size 1 1) (thickness 0.25)))
+  )
+  (gr_text "RF Noise Raspberry Hat V1.0" (at 78.0415 32.512) (layer F.SilkS)
+    (effects (font (size 1 1) (thickness 0.25)))
+  )
+  (gr_text "Giga Technology" (at 73.787 30.099) (layer F.Cu)
+    (effects (font (size 1 1) (thickness 0.25)))
+  )
   (gr_line (start 34.5 77.5) (end 46.9 77.5) (angle 90) (layer Edge.Cuts) (width 0.15))
   (gr_line (start 34 77.5) (end 34.5 77.5) (angle 90) (layer Edge.Cuts) (width 0.15))
@@
   (gr_arc (start 32 24) (end 29 24) (angle 90) (layer Edge.Cuts) (width 0.15))
   (gr_line (start 32 21) (end 90 21) (angle 90) (layer Edge.Cuts) (width 0.15))
+  (segment (start 42.45 23.73) (end 42.45 24.1615) (width 0.4) (layer F.Cu) (net 1))
+  (segment (start 42.45 24.1615) (end 41.275 25.3365) (width 0.4) (layer F.Cu) (net 1))
+  (segment (start 43.0345 28.1305) (end 44.384 29.48) (width 0.4) (layer F.Cu) (net 1))
+  (segment (start 42.037 28.1305) (end 43.0345 28.1305) (width 0.4) (layer F.Cu) (net 1))
+  (segment (start 41.275 27.3685) (end 42.037 28.1305) (width 0.4) (layer F.Cu) (net 1))
+  (segment (start 41.275 25.3365) (end 41.275 27.3685) (width 0.4) (layer F.Cu) (net 1))
   (segment (start 58.166 37.084) (end 58.166 37.4015) (width 0.4) (layer F.Cu) (net 1))
   (via (at 64.262 40.386) (size 0.889) (drill 0.381) (layers F.Cu B.Cu) (net 1))
@@
   (segment (start 50.8635 39.0525) (end 52.7685 39.0525) (width 0.5) (layer B.Cu) (net 1))
   (segment (start 44.384 29.48) (end 44.339 29.48) (width 0.5) (layer F.Cu) (net 1))
-  (segment (start 44.339 29.48) (end 42.291 27.432) (width 0.5) (layer F.Cu) (net 1))
-  (segment (start 42.291 27.432) (end 41.529 27.432) (width 0.5) (layer F.Cu) (net 1))
-  (segment (start 41.529 27.432) (end 41.275 27.178) (width 0.5) (layer F.Cu) (net 1))
-  (segment (start 41.275 27.178) (end 41.275 24.905) (width 0.5) (layer F.Cu) (net 1))
-  (segment (start 41.275 24.905) (end 42.45 23.73) (width 0.5) (layer F.Cu) (net 1))
   (segment (start 61.468 62.042) (end 61.468 58.594) (width 0.5) (layer F.Cu) (net 1))
   (segment (start 61.468 58.594) (end 59.516 56.642) (width 0.5) (layer F.Cu) (net 1))
@@
   (segment (start 66.802 38.782) (end 66.802 36.088) (width 1.25) (layer F.Cu) (net 2))
   (segment (start 66.802 36.088) (end 66.782 36.068) (width 1.25) (layer F.Cu) (net 2))
-  (segment (start 56.576 36.434) (end 59.832 36.434) (width 0.4) (layer F.Cu) (net 3))
-  (segment (start 59.832 36.434) (end 60.198 36.068) (width 0.4) (layer F.Cu) (net 3))
-  (segment (start 60.198 36.068) (end 64.282 36.068) (width 0.4) (layer F.Cu) (net 3))
+  (segment (start 56.576 36.434) (end 57.1015 36.434) (width 0.4) (layer F.Cu) (net 3))
+  (segment (start 61.468 36.068) (end 64.282 36.068) (width 0.4) (layer F.Cu) (net 3))
+  (segment (start 61.2775 36.2585) (end 61.468 36.068) (width 0.4) (layer F.Cu) (net 3))
+  (segment (start 57.277 36.2585) (end 61.2775 36.2585) (width 0.4) (layer F.Cu) (net 3))
+  (segment (start 57.1015 36.434) (end 57.277 36.2585) (width 0.4) (layer F.Cu) (net 3))
   (segment (start 62.118 62.042) (end 66.716 62.042) (width 0.4) (layer F.Cu) (net 4))
   (segment (start 66.716 62.042) (end 66.802 61.956) (width 0.4) (layer F.Cu) (net 4))
@@
   (segment (start 40.4495 38.354) (end 39.5135 37.418) (width 1.25) (layer F.Cu) (net 18))
   (segment (start 39.5135 37.418) (end 37.592 37.418) (width 1.25) (layer F.Cu) (net 18))
-  (segment (start 35.248 38.924) (end 35.248 36.5815) (width 0.4) (layer B.Cu) (net 19) (status 400000))
+  (segment (start 44.45 43.688) (end 44.45 46.101) (width 0.4) (layer F.Cu) (net 19))
+  (via (at 45.6565 55.0545) (size 0.889) (drill 0.381) (layers F.Cu B.Cu) (net 19))
+  (segment (start 45.6565 53.1495) (end 45.6565 55.0545) (width 0.4) (layer B.Cu) (net 19))
+  (via (at 45.6565 53.1495) (size 0.889) (drill 0.381) (layers F.Cu B.Cu) (net 19))
+  (segment (start 45.6565 50.9905) (end 45.6565 53.1495) (width 0.4) (layer F.Cu) (net 19))
+  (via (at 45.6565 50.9905) (size 0.889) (drill 0.381) (layers F.Cu B.Cu) (net 19))
+  (segment (start 45.6565 48.7045) (end 45.6565 50.9905) (width 0.4) (layer B.Cu) (net 19))
+  (via (at 45.6565 48.7045) (size 0.889) (drill 0.381) (layers F.Cu B.Cu) (net 19))
+  (segment (start 45.6565 46.99) (end 45.6565 48.7045) (width 0.4) (layer F.Cu) (net 19))
+  (segment (start 45.847 46.7995) (end 45.6565 46.99) (width 0.4) (layer F.Cu) (net 19))
+  (via (at 45.847 46.7995) (size 0.889) (drill 0.381) (layers F.Cu B.Cu) (net 19))
+  (segment (start 47.4345 46.7995) (end 45.847 46.7995) (width 0.4) (layer B.Cu) (net 19))
+  (via (at 47.4345 46.7995) (size 0.889) (drill 0.381) (layers F.Cu B.Cu) (net 19))
+  (segment (start 47.4345 48.5775) (end 47.4345 46.7995) (width 0.4) (layer F.Cu) (net 19))
+  (via (at 47.4345 48.5775) (size 0.889) (drill 0.381) (layers F.Cu B.Cu) (net 19))
+  (segment (start 47.4345 50.419) (end 47.4345 48.5775) (width 0.4) (layer B.Cu) (net 19))
+  (via (at 47.4345 50.419) (size 0.889) (drill 0.381) (layers F.Cu B.Cu) (net 19))
+  (segment (start 47.4345 52.197) (end 47.4345 50.419) (width 0.4) (layer F.Cu) (net 19))
+  (via (at 47.4345 52.197) (size 0.889) (drill 0.381) (layers F.Cu B.Cu) (net 19))
+  (segment (start 47.4345 53.975) (end 47.4345 52.197) (width 0.4) (layer B.Cu) (net 19))
+  (via (at 47.4345 53.975) (size 0.889) (drill 0.381) (layers F.Cu B.Cu) (net 19))
+  (segment (start 47.4345 55.626) (end 47.4345 53.975) (width 0.4) (layer F.Cu) (net 19))
+  (via (at 47.4345 55.626) (size 0.889) (drill 0.381) (layers F.Cu B.Cu) (net 19))
+  (segment (start 47.4345 57.0865) (end 47.4345 55.626) (width 0.4) (layer B.Cu) (net 19))
+  (via (at 47.4345 57.0865) (size 0.889) (drill 0.381) (layers F.Cu B.Cu) (net 19))
+  (segment (start 45.4025 57.0865) (end 47.4345 57.0865) (width 0.4) (layer F.Cu) (net 19))
+  (via (at 45.4025 57.0865) (size 0.889) (drill 0.381) (layers F.Cu B.Cu) (net 19))
+  (segment (start 43.561 57.0865) (end 45.4025 57.0865) (width 0.4) (layer B.Cu) (net 19))
+  (via (at 43.561 57.0865) (size 0.889) (drill 0.381) (layers F.Cu B.Cu) (net 19))
+  (segment (start 43.561 55.0545) (end 43.561 57.0865) (width 0.4) (layer F.Cu) (net 19))
+  (via (at 43.561 55.0545) (size 0.889) (drill 0.381) (layers F.Cu B.Cu) (net 19))
+  (segment (start 43.561 52.07) (end 43.561 55.0545) (width 0.4) (layer B.Cu) (net 19))
+  (via (at 43.561 52.07) (size 0.889) (drill 0.381) (layers F.Cu B.Cu) (net 19))
+  (segment (start 43.561 49.3395) (end 43.561 52.07) (width 0.4) (layer F.Cu) (net 19))
+  (via (at 43.561 49.3395) (size 0.889) (drill 0.381) (layers F.Cu B.Cu) (net 19))
+  (segment (start 43.561 46.99) (end 43.561 49.3395) (width 0.4) (layer B.Cu) (net 19))
+  (via (at 43.561 46.99) (size 0.889) (drill 0.381) (layers F.Cu B.Cu) (net 19))
+  (segment (start 44.45 46.101) (end 43.561 46.99) (width 0.4) (layer F.Cu) (net 19))
+  (segment (start 45.974 37.084) (end 43.7515 37.084) (width 0.4) (layer F.Cu) (net 19))
+  (via (at 41.3385 36.576) (size 0.889) (drill 0.381) (layers F.Cu B.Cu) (net 19))
+  (segment (start 43.2435 36.576) (end 41.3385 36.576) (width 0.4) (layer B.Cu) (net 19))
+  (via (at 43.2435 36.576) (size 0.889) (drill 0.381) (layers F.Cu B.Cu) (net 19))
+  (segment (start 43.7515 37.084) (end 43.2435 36.576) (width 0.4) (layer F.Cu) (net 19))
+  (segment (start 35.2425 32.131) (end 38.0365 32.131) (width 0.4) (layer F.Cu) (net 19))
+  (via (at 38.0365 32.131) (size 0.889) (drill 0.381) (layers F.Cu B.Cu) (net 19))
+  (segment (start 35.248 38.924) (end 35.248 36.5815) (width 0.4) (layer B.Cu) (net 19))
   (via (at 35.179 36.5125) (size 0.889) (drill 0.381) (layers F.Cu B.Cu) (net 19))
   (segment (start 35.248 36.5815) (end 35.179 36.5125) (width 0.4) (layer B.Cu) (net 19))
@@
     (polygon
       (pts
-        (xy 48.13257 77.279506) (xy 28.829 77.5335) (xy 28.829 21.1455) (xy 48.006 21.1455)
-      )
-    )
-  )
-  (zone (net 19) (net_name GNDA) (layer F.Cu) (hatch edge 0.508)
-    (connect_pads (clearance 0.508))
-    (min_thickness 0.254)
-    (fill yes (arc_segments 16) (thermal_gap 0.508) (thermal_bridge_width 0.508))
-    (polygon
-      (pts
-        (xy 48.133 77.47) (xy 48.13257 77.279506) (xy 48.133 77.2795)
+        (xy 48.0695 49.307856) (xy 48.0695 42.545) (xy 52.2605 42.545) (xy 52.2605 77.47) (xy 48.0695 77.47)
+        (xy 48.0695 77.280336) (xy 28.829 77.5335) (xy 28.829 21.1455) (xy 48.006 21.1455)
       )
     )
@@
       )
     )
+  )
+  (zone (net 0) (net_name "") (layer F.Cu) (hatch edge 0.508)
+    (connect_pads (clearance 0.508))
+    (min_thickness 0.254)
+    (keepout (tracks not_allowed) (vias not_allowed) (copperpour allowed))
+    (fill (arc_segments 16) (thermal_gap 0.508) (thermal_bridge_width 0.508))
+    (polygon
+      (pts
+        (xy 28.829 21.1455) (xy 28.829 28.067) (xy 28.956 28.067)
+      )
+    )

Commit message: Fix Transistor pin config
Parts:
- Q1, Q2: value BC817 -> BC847
Connections:
- Q1 pad 1: GND -> Net-(Q1-Pad1)
- Q1 pad 2: Net-(Q1-Pad2) -> GND
- Q2 pad 1: GND -> Net-(Q2-Pad1)
- Q2 pad 2: Net-(Q2-Pad2) -> GND
- R3 pad 2: Net-(Q1-Pad2) -> Net-(Q1-Pad1)
- R5 pad 1: Net-(Q2-Pad2) -> Net-(Q2-Pad1)
Routing:
- net GND: track 409.5 -> 396.5 mm, vias 41 -> 42
- net Net-(Q2-Pad1): track 0.00 -> 8.77 mm
- net Net-(Q1-Pad1): track 0.00 -> 5.78 mm
- net Net-(Q2-Pad2): track 3.62 -> 0.00 mm
- net Net-(Q1-Pad2): track 3.58 -> 0.00 mm

Commit message: adding V2 files
Other:
- board text added: "FIX SMA Connector"
Changed lines of the file:
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@@
     (links 92)
     (no_connects 0)
-    (area 28.924999 20.924999 94.075001 77.575001)
+    (area 16.276381 15.477 95.55962 87.217001)
     (thickness 1.6)
-    (drawings 41)
+    (drawings 42)
     (tracks 420)
     (zones 0)
@@
       (drillshape 0)
       (scaleselection 1)
-      (outputdirectory gerber/))
+      (outputdirectory Gerber_manufacture/))
   )
   (net 0 "")
@@
       (effects (font (size 1 1) (thickness 0.15)))
     )
-    (fp_text value Conn_Coaxial (at -8.382 0.254 180) (layer F.Fab)
+    (fp_text value Conn_Coaxial (at 2.54 -40.005 180) (layer F.Fab)
       (effects (font (size 1 1) (thickness 0.15)))
     )
@@
       (effects (font (size 1 1) (thickness 0.15)))
     )
-    (fp_text value Conn_01x03 (at 3.81 8.636) (layer F.Fab)
+    (fp_text value Conn_01x03 (at -18.796 0.889) (layer F.Fab)
       (effects (font (size 1 1) (thickness 0.15)))
     )
@@
       (effects (font (size 1 1) (thickness 0.15)))
     )
-    (fp_text value Conn_01x01 (at -0.242 6.264) (layer F.Fab)
+    (fp_text value Conn_01x01 (at -11.164 0.93) (layer F.Fab)
       (effects (font (size 1 1) (thickness 0.15)))
     )
@@
       (effects (font (size 1 1) (thickness 0.15)))
     )
-    (fp_text value Conn_01x01 (at 0 4.2) (layer F.Fab)
+    (fp_text value Conn_01x01 (at -70.053 -7.325) (layer F.Fab)
       (effects (font (size 1 1) (thickness 0.15)))
     )
@@
     (descr "Mounting Hole 3.2mm, no annular, M3")
     (tags "mounting hole 3.2mm no annular m3")
-    (fp_text reference H3 (at 0 -4.2) (layer F.SilkS)
+    (fp_text reference H3 (at -2.02 2.94) (layer F.SilkS)
       (effects (font (size 1 1) (thickness 0.15)))
     )
@@
       (effects (font (size 1 1) (thickness 0.15)))
     )
-    (fp_text value Conn_01x01 (at 10.338 -0.362) (layer F.Fab)
+    (fp_text value Conn_01x01 (at -71.069 38.627) (layer F.Fab)
       (effects (font (size 1 1) (thickness 0.15)))
     )
@@
     )
   )
+  (gr_text "FIX SMA Connector" (at 104.267 43.18) (layer F.Cu)
+    (effects (font (size 1 1) (thickness 0.25)))
+  )
   (gr_text http://www.giga.co.za (at 83.7565 37.6555) (layer F.SilkS)
