File: rf_noise_antenna_v2.sch (KiCad schematic (older format))
At the start: 60 parts, among them J1 Conn_Coaxial, J2 Conn_Coaxial, J3 Conn_01x03, J4 Raspberry_Pi_2_3, J5 SMA Edge, K1 MASWSS0115, K2 MASWSS0115, Q1 BC847, Q2 BC847, Q3 BFQ149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

Commit message: adding V2 files
Parts:
- removed AE1: Antenna, symbol Antenna
- removed C16: 22uF, Capacitors_Tantalum_SMD:CP_Tantalum_Case-C_EIA-6032-28_Hand, symbol CP
- removed C17, C19: 100nF, Capacitors_SMD:C_0805_HandSoldering, symbol C
- removed C18: 470nF Foil, Capacitors_SMD:C_0805_HandSoldering, symbol C
- removed H5: Conn_01x01, Mounting_Holes:MountingHole_3.2mm_M3, symbol Conn_01x01
- removed J5: SMA Edge, Connectors_Molex:Molex_SMA_Jack_Edge_Mount, symbol Conn_Coaxial
- removed L7: 8 Turns BN73-202, rf_noise_antenna:BN73-202_Ferrite_Balun, symbol L
- removed L8: 5Turns BN43-2402, rf_noise_antenna:BN43-2402_Ferrite_Balun, symbol L
- removed Q3: BFQ149, TO_SOT_Packages_SMD:SOT-89-3_Handsoldering, symbol 2N3905
- removed Q4: BF862, TO_SOT_Packages_SMD:SOT-23, symbol Q_NJFET_DGS
- removed R10: 10M, Resistors_SMD:R_0805_HandSoldering, symbol R
- removed R11, R8: 1M, Resistors_SMD:R_0805_HandSoldering, symbol R
- removed R12: 100 0.5W, Resistors_SMD:R_1206_HandSoldering, symbol R
- removed R7, R9: 100, Resistors_SMD:R_0805_HandSoldering, symbol R
- J1, J2: footprint Connectors_Molex:Molex_SMA_Jack_Edge_Mount -> Bacar:SMA_Edge
Connections:
- net labels removed: GNDPWR
- wire segments 132 -> 105
Other:
- note removed: "12V"
- note removed: "Block FM 88-108Mhz"
- note removed: "Heatsink"
- note removed: "Prevent VHF\nOselation"
- note removed: "To Do\n\n1) Check transistor pins\n2) Add Unductor Package details"
